Commit message: Add: 添加深度相机及模型

File: robots/mpo_700/urdf/mpo_700_body.urdf.xacro (robot description, xacro)
@@ -1,4 +1,10 @@
 <?xml version="1.0"?>
 <robot xmlns:xacro="http://www.ros.org/wiki/xacro" name="mpo_700">
+    <!-- Depth camera visual pose tuning (affects only mesh appearance, not TF/sensor) -->
+    <xacro:property name="depth_cam_visual_xyz" value="0 0 0"/>
+    <!-- Default: pitch -90deg (about Y) and yaw +90deg (about Z), lens faces +X and body horizontal -->
+    <!-- <xacro:property name="depth_cam_visual_rpy" value="0 -1.57079632679 1.57079632679"/> -->
+    <!-- 相机gui正确,点云错误 -->
+    <xacro:property name="depth_cam_visual_rpy" value="1.57079632679 0 1.57079632679"/>
     <link name="base_footprint"/>
     <link name="base_link">
@@ -176,3 +182,40 @@
         </xacro:docking_adapter>
     </xacro:if>
+    <!-- Depth camera mounting (front top center) -->
+    <joint name="depth_camera_joint" type="fixed">
+        <parent link="base_link"/>
+        <!-- Slightly in front and above the base; looking forward -->
+        <origin xyz="0.35 0.0 0.25" rpy="0 0 0"/>
+        <child link="depth_camera_link"/>
+    </joint>
+    <link name="depth_camera_link">
+        <inertial>
+            <mass value="0.5"/>
+            <origin xyz="0 0 0" rpy="0 0 0"/>
+            <inertia ixx="0.002" ixy="0" ixz="0" iyy="0.002" iyz="0" izz="0.002"/>
+        </inertial>
+        <visual>
+            <!-- Mesh-only pose: can be tuned with depth_cam_visual_xyz/rpy without touching TF/sensor -->
+            <origin xyz="${depth_cam_visual_xyz}" rpy="${depth_cam_visual_rpy}"/>
+            <geometry>
+                <mesh filename="package://neo_simulation2/components/meshes/d435.dae" scale="1 1 1"/>
+            </geometry>
+        </visual>
+        <collision>
+            <origin xyz="${depth_cam_visual_xyz}" rpy="${depth_cam_visual_rpy}"/>
+            <geometry>
+                <mesh filename="package://neo_simulation2/components/meshes/d435.dae" scale="1 1 1"/>
+            </geometry>
+        </collision>
+    </link>
+    <!-- Depth camera optical frame (standard optical: x right, y down, z forward) -->
+    <joint name="depth_camera_optical_joint" type="fixed">
+        <parent link="depth_camera_link"/>
+        <!-- REP 103 / optical frames: rotate from robot-forward (x forward, z up) to optical (z forward, x right, y down) -->
+        <!-- <origin xyz="0 0 0" rpy="1.57079632679 0 1.57079632679"/> -->
+        <origin xyz="0 0 0" rpy="-1.57079632679 0 -1.57079632679"/>
+        <!-- <origin xyz="0 0 0" rpy=".0 0 0"/> -->
+        <child link="depth_camera_optical_frame"/>
+    </joint>
+    <link name="depth_camera_optical_frame"/>
 </robot>

File: robots/mpo_700/urdf/mpo_700_gazebo.urdf.xacro (robot description, xacro)
@@ -3,4 +3,5 @@
     <!-- Include macros -->
     <xacro:include filename="$(find neo_simulation2)/components/common_macro/gazebo_lidar_macro.xacro" />
+    <xacro:include filename="$(find neo_simulation2)/components/common_macro/gazebo_depth_camera_macro.xacro" />
     <xacro:include filename="$(find neo_simulation2)/components/common_macro/gazebo_object_controller_macro.xacro" />
     <xacro:include filename="$(find neo_simulation2)/robots/mpo_700/urdf/macro/gazebo_mpo_700_wheel_macro.xacro" />
@@ -64,3 +65,19 @@
     <!-- <xacro:include filename="$(find neo_simulation2)/robots/mpo_700/xacros/sick_S300.xacro" /> -->
     <!--Ultrasonics, cameras and IMU's  -->
+    <!-- Depth camera sensor instantiation -->
+    <xacro:gazebo_depth_camera_sensor
+        sensor_name="front_depth_camera"
+        link_name="depth_camera_link"
+        frame_name="depth_camera_optical_frame"
+        update_rate="15"
+        width="640"
+        height="480"
+        fov="1.0472"
+        near_clip="0.1"
+        far_clip="10.0"
+        image_topic="/camera/depth/image_raw"
+        info_topic="/camera/depth/camera_info"
+        points_topic="/camera/points"
+        visualize="false"
+    />
 </robot>
